Commit message: 添加stl文件及base_footprint

File: src/urdf_1/urdf/urdf_1.urdf (robot description, URDF)
Before this commit: robot urdf_1, 11 links, 10 joints
Links:
- added link base_footprint, mass 0; collision mesh filename=package://urdf_1/meshes/base_footprint.STL
Joints:
- added joint joint_name: type fixed, parent base_footprint, child base_link, origin xyz=0.0 0.0 0.145 rpy=0.0 0.0 0.0, axis 0.0 0.0 0.0, limit lower=0.0 upper=0.0 effort=0.0 velocity=0.0
