Commit message: 添加雷达

File: src/urdf/urdf/urdf_1.urdf (robot description, URDF)
Before this commit: robot urdf_1, 12 links, 11 joints
Joints:
- joint Joint_laser: origin xyz=0 0.48 0.0275 rpy=1.5708 0 0 -> xyz=0 0.48 0.0275 rpy=0 0 -1.5708

Commit message: 创建地图

File: src/urdf/urdf/urdf_1.urdf (robot description, URDF)
Before this commit: robot urdf_1, 12 links, 11 joints
Links:
- removed link Link_laser
- added link laser_link, mass 0.201875516239374; collision mesh filename=package://car_description/meshes/laser_link.STL; visual mesh filename=package://car_description/meshes/laser_link.STL
Joints:
- joint Joint_laser: child Link_laser -> laser_link
