Commit message: 修改URDF的TF

File: src/urdf/urdf/car_arm_urdf_2.0.urdf (robot description, URDF)
Before this commit: robot car_arm_urdf, 22 links, 21 joints
Links:
- link L_wheel_link: geometry collision mesh filename=package://car_description/meshes/arm/L_wheel_link.STL; visual mesh filename=package://car_description/meshes/arm/L_wheel_link.STL
- link R_wheel_link: geometry collision mesh filename=package://car_description/meshes/arm/R_wheel_link.STL; visual mesh filename=package://car_description/meshes/arm/R_wheel_link.STL
- link arm_1_link: geometry collision mesh filename=package://car_description/meshes/arm/arm_1_link.STL; visual mesh filename=package://car_description/meshes/arm/arm_1_link.STL
- link arm_2_link: geometry collision mesh filename=package://car_description/meshes/arm/arm_2_link.STL; visual mesh filename=package://car_description/meshes/arm/arm_2_link.STL
- link arm_3_link: geometry collision mesh filename=package://car_description/meshes/arm/arm_3_link.STL; visual mesh filename=package://car_description/meshes/arm/arm_3_link.STL
- link arm_4_link: geometry collision mesh filename=package://car_description/meshes/arm/arm_4_link.STL; visual mesh filename=package://car_description/meshes/arm/arm_4_link.STL
- link arm_5_link: geometry collision mesh filename=package://car_description/meshes/arm/arm_5_link.STL; visual mesh filename=package://car_description/meshes/arm/arm_5_link.STL
- link arm_base_link: geometry collision mesh filename=package://car_description/meshes/arm/arm_base_link.STL; visual mesh filename=package://car_description/meshes/arm/arm_base_link.STL
- link arm_camera_link: mass 0.000379351096233468 -> 0.000379351096233471; geometry collision mesh filename=package://car_description/meshes/arm/arm_camera_link.STL; visual mesh filename=package://car_description/meshes/arm/arm_camera_link.STL
- link back_shell_link: mass 0.695304748322187 -> 0.695304748320442; geometry collision mesh filename=package://car_description/meshes/arm/back_shell_link.STL; visual mesh filename=package://car_description/meshes/arm/back_shell_link.STL
- link base_link: geometry collision mesh filename=package://car_description/meshes/arm/base_link.STL; visual mesh filename=package://car_description/meshes/arm/base_link.STL
- link battery_link: geometry collision mesh filename=package://car_description/meshes/arm/battery_link.STL; visual mesh filename=package://car_description/meshes/arm/battery_link.STL
- link camera_1_link: geometry collision mesh filename=package://car_description/meshes/arm/camera_1_link.STL; visual mesh filename=package://car_description/meshes/arm/camera_1_link.STL
- link camera_2_link: geometry collision mesh filename=package://car_description/meshes/arm/camera_2_link.STL; visual mesh filename=package://car_description/meshes/arm/camera_2_link.STL
- link clamp_left_link: mass 26.7299172136853 -> 0.0138851667711793; geometry collision mesh filename=package://car_description/meshes/arm/clamp_left_link.STL; visual mesh filename=package://car_description/meshes/arm/clamp_left_link.STL
- link clamp_right_link: mass 0.0138851667711794 -> 0.0138851667711793; geometry collision mesh filename=package://car_description/meshes/arm/clamp_right_link.STL; visual mesh filename=package://car_description/meshes/arm/clamp_right_link.STL
- link front_shell_link: mass 0.757865823241688 -> 0.757865840617367; geometry collision mesh filename=package://car_description/meshes/arm/front_shell_link.STL; visual mesh filename=package://car_description/meshes/arm/front_shell_link.STL
- link imu_link: geometry collision mesh filename=package://car_description/meshes/arm/imu_link.STL; visual mesh filename=package://car_description/meshes/arm/imu_link.STL
- link laser_link: geometry collision mesh filename=package://car_description/meshes/arm/laser_link.STL; visual mesh filename=package://car_description/meshes/arm/laser_link.STL
- link middle_shell_link: mass 0.376095918062655 -> 0.376095918062654; geometry collision mesh filename=package://car_description/meshes/arm/middle_shell_link.STL; visual mesh filename=package://car_description/meshes/arm/middle_shell_link.STL
- link pole_link: geometry collision mesh filename=package://car_description/meshes/arm/pole_link.STL; visual mesh filename=package://car_description/meshes/arm/pole_link.STL
- link up_shell_link: geometry collision mesh filename=package://car_description/meshes/arm/up_shell_link.STL; visual mesh filename=package://car_description/meshes/arm/up_shell_link.STL
Joints:
- joint arm_2_joint: axis 0 0 0 -> 0 1 0; origin xyz=-0.035 0 0.07 rpy=0 0 0 -> xyz=-0.0349999999999994 0 0.0700000000000004 rpy=0 0 0
- joint arm_3_joint: origin xyz=-0.0045 0 0.0305 rpy=0 0 0 -> xyz=-0.00449999999999967 0 0.0305 rpy=0 0 0
- joint arm_4_joint: origin xyz=0.092971 0 -0.010704 rpy=0 0.63688 0 -> xyz=0.0965000000000001 0 0 rpy=0 0 0
- joint arm_5_joint: origin xyz=0.0375 0 0 rpy=-0.043872 0 0 -> xyz=0.0375 0 0 rpy=0 0 0
- joint arm_camera_joint: origin xyz=0.00349999999999812 0 0 rpy=0 0 0 -> xyz=0.0035 0 0 rpy=0 0 0
- joint clamp_left_joint: origin xyz=0.004 0.01 0 rpy=0 0 0 -> xyz=0.004 0.035 0 rpy=0 0 0
- joint clamp_right_joint: origin xyz=0.004 -0.01 0 rpy=0 0 0 -> xyz=0.004 -0.035 0 rpy=0 0 0
- joint pole_joint: axis -1 0 0 -> 0 1 0

File: src/urdf/urdf/car_urdf.urdf (robot description, URDF)
Before this commit: robot car_urdf, 16 links, 15 joints
Links:
- added link arm_1_link, mass 0.143863120805872; collision mesh filename=package://car_description/meshes/arm/arm_1_link.STL; visual mesh filename=package://car_description/meshes/arm/arm_1_link.STL
- added link arm_2_link, mass 0.186614834092236; collision mesh filename=package://car_description/meshes/arm/arm_2_link.STL; visual mesh filename=package://car_description/meshes/arm/arm_2_link.STL
- added link arm_3_link, mass 0.16931961826588; collision mesh filename=package://car_description/meshes/arm/arm_3_link.STL; visual mesh filename=package://car_description/meshes/arm/arm_3_link.STL
- added link arm_4_link, mass 0.051853364801175; collision mesh filename=package://car_description/meshes/arm/arm_4_link.STL; visual mesh filename=package://car_description/meshes/arm/arm_4_link.STL
- added link arm_5_link, mass 0.0303242029391938; collision mesh filename=package://car_description/meshes/arm/arm_5_link.STL; visual mesh filename=package://car_description/meshes/arm/arm_5_link.STL
- added link arm_base_link, mass 0.0597062822264354; collision mesh filename=package://car_description/meshes/arm/arm_base_link.STL; visual mesh filename=package://car_description/meshes/arm/arm_base_link.STL
- added link arm_camera_link, mass 0.000379351096233471; collision mesh filename=package://car_description/meshes/arm/arm_camera_link.STL; visual mesh filename=package://car_description/meshes/arm/arm_camera_link.STL
- added link clamp_left_link, mass 0.0138851667711793; collision mesh filename=package://car_description/meshes/arm/clamp_leftlink.STL; visual mesh filename=package://car_description/meshes/arm/clamp_leftlink.STL
- added link clamp_right_link, mass 0.0138851667711793; collision mesh filename=package://car_description/meshes/arm/clamp_right_link.STL; visual mesh filename=package://car_description/meshes/arm/clamp_right_link.STL
Joints:
- added joint arm_1_joint: type revolute, parent arm_base_link, child arm_1_link, origin xyz=0 0 0 rpy=0 0 0, axis 0 0 -1, limit lower=0 upper=3.14 effort=0 velocity=0
- added joint arm_2_joint: type revolute, parent arm_1_link, child arm_2_link, origin xyz=0.03 0 0.07 rpy=0 0 0, axis 0 1 0, limit lower=0 upper=0 effort=0 velocity=0
- added joint arm_3_joint: type revolute, parent arm_2_link, child arm_3_link, origin xyz=-0.118 0 0.0305 rpy=0 0 0, axis 0 1 0, limit lower=0 upper=3.14 effort=0 velocity=0
- added joint arm_4_joint: type revolute, parent arm_3_link, child arm_4_link, origin xyz=0.127 0 0 rpy=0 0 0, axis 0 1 0, limit lower=0 upper=1.57 effort=0 velocity=0
- added joint arm_5_joint: type revolute, parent arm_4_link, child arm_5_link, origin xyz=0.0555 0 0 rpy=0 0 0, axis 1 0 0, limit lower=-3.14 upper=3.14 effort=0 velocity=0
- added joint arm_base_joint: type prismatic, parent base_link, child arm_base_link, origin xyz=0.3465 0 -0.0225 rpy=0 0 0, axis 0 1 0, limit lower=-0.12 upper=0.12 effort=0 velocity=0
- added joint arm_camera_joint: type fixed, parent arm_5_link, child arm_camera_link, origin xyz=0.0035 0 0 rpy=0 0 0, axis 0 0 0
- added joint clamp_left_joint: type prismatic, parent arm_5_link, child clamp_left_link, origin xyz=0.004 0.01 0 rpy=0 0 0, axis 0 -1 0, limit lower=0 upper=0.025 effort=0 velocity=0
- added joint clamp_right_joint: type prismatic, parent arm_5_link, child clamp_right_link, origin xyz=0.004 -0.01 0 rpy=0 0 0, axis 0 1 0, limit lower=0 upper=0.025 effort=0 velocity=0
