Commit message: gazebo中能够正常遥控

File: src/urdf/urdf/car_urdf.urdf (robot description, URDF)
Before this commit: robot car_urdf, 16 links, 15 joints
Links:
- link B_caster_link: mass 0.0 -> 0.005
- link F_caster_link: mass 0.0 -> 0.005
- link L_wheel_link: geometry collision cylinder length=0.044 radius=0.097; visual mesh filename=package://car_description/meshes/L_wheel_link.STL
- link R_wheel_link: geometry collision cylinder length=0.044 radius=0.097; visual mesh filename=package://car_description/meshes/R_wheel_link.STL
Joints:
- removed joint L_wheel_link
- added joint L_wheel_joint: type continuous, parent base_link, child L_wheel_link, origin xyz=0 0.143 0 rpy=0 0 0, axis 0 -1 0
- joint B_caster_joint: origin xyz=-0.2 0.0 -0.077 rpy=0.0 0.0 0.0 -> xyz=-0.2 0.0 -0.0765 rpy=0.0 0.0 0.0
- joint F_caster_joint: origin xyz=0.2 0.0 -0.077 rpy=0.0 0.0 0.0 -> xyz=0.2 0.0 -0.0765 rpy=0.0 0.0 0.0
- joint joint_name: origin xyz=0.0 0.0 0.0969 rpy=0.0 0.0 0.0 -> xyz=0.0 0.0 0.097 rpy=0.0 0.0 0.0
- joint laser_joint: origin xyz=0.155 0 0.2055 rpy=0 0 0 -> xyz=0.155 0 0.1855 rpy=0 0 3.14
- joint pole_joint: type continuous -> fixed

Commit message: URDF修改限位

File: src/urdf/urdf/car_urdf.urdf (robot description, URDF)
Before this commit: robot car_urdf, 25 links, 24 joints
Joints:
- joint arm_1_joint: limit lower=0 upper=3.14 effort=0 velocity=0 -> lower=-1.55 upper=1.55 effort=0 velocity=0
- joint arm_2_joint: limit lower=0 upper=0 effort=0 velocity=0 -> lower=0 upper=3.14 effort=0 velocity=0
- joint arm_3_joint: limit lower=0 upper=3.14 effort=0 velocity=0 -> lower=-3.14 upper=0.04 effort=0 velocity=0
- joint arm_4_joint: limit lower=0 upper=1.57 effort=0 velocity=0 -> lower=-1.8 upper=1.8 effort=0 velocity=0
- joint clamp_left_joint: limit lower=0 upper=0.025 effort=0 velocity=0 -> lower=-0.035 upper=0 effort=0 velocity=0
- joint clamp_right_joint: limit lower=0 upper=0.025 effort=0 velocity=0 -> lower=-0.035 upper=0 effort=0 velocity=0

Commit message: task初步-2

File: src/urdf/urdf/car_urdf.urdf (robot description, URDF)
Before this commit: robot car_urdf, 25 links, 24 joints
Joints:
- joint arm_base_joint: axis 0 1 0 -> (none); limit lower=-0.12 upper=0.12 effort=0 velocity=0 -> (none); type prismatic -> fixed

Commit message: fix: align task integration with add_arm

File: src/urdf/urdf/car_urdf.urdf (robot description, URDF)
Before this commit: robot car_urdf, 25 links, 24 joints
Joints:
- joint arm_base_joint: axis (none) -> 0 1 0; limit (none) -> lower=-0.12 upper=0.12 effort=0 velocity=0; type fixed -> prismatic

Commit message: 更改参数适配实车

File: src/urdf/urdf/car_urdf.urdf (robot description, URDF)
Before this commit: robot car_urdf, 25 links, 24 joints
Links:
- removed link laser_link
- added link laser, mass 0.04345685683984; collision mesh filename=package://car_description/meshes/laser_link.STL; visual mesh filename=package://car_description/meshes/laser_link.STL
Joints:
- joint laser_joint: child laser_link -> laser; origin xyz=0.155 0 0.1855 rpy=0 0 3.14 -> xyz=-0.06 0.0 0.0475 rpy=0 0 0
